File: hardware/PCB_35x25_4Vueltas/NFC_Programmer.kicad_sch (KiCad schematic)
At the start: 41 parts, among them J1 Conn_01x08, J2 Conn_01x02_Pin, U1 MFRC63002HN,151, Y1 Crystal_GND23

Commit message: Actualizacion
Parts:
- removed Y1: Crystal_GND23, Crystal:Crystal_SMD_2016-4Pin_2.0x1.6mm, symbol Device:Crystal_GND23
- added J3: Conn_01x02_Pin, Connector_PinHeader_2.54mm:PinHeader_1x02_P2.54mm_Vertical, symbol Connector:Conn_01x02_Pin
- added Y1: Crystal_27.12MHz, Crystal:Crystal_SMD_2016-4Pin_2.0x1.6mm, symbol Device:Crystal_GND24
- C14: value C -> TBD
- J1: footprint Connector_PinHeader_2.00mm:PinHeader_1x08_P2.00mm_Vertical -> Connector_PinHeader_2.54mm:PinHeader_1x08_P2.54mm_Vertical
- J2: footprint Connector_PinHeader_2.00mm:PinHeader_1x02_P2.00mm_Vertical -> Connector_PinHeader_2.54mm:PinHeader_1x02_P2.54mm_Vertical
Connections:
- net GND: now also Y1.2, Y1.4
- net TX1: now also J3.1 (Pin_1)
- net TX2: now also J3.2 (Pin_2)
- net at C7.1, U1.19 (XTAL1): now also Y1.1
- net at C8.1, U1.20 (XTAL2): now also Y1.3
Changed lines of the file:
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@@
+    (stroke (width 0) (type default))
+  )
+  (wire (pts (xy 154.6098 73.5838) (xy 156.21 73.5838))
     (stroke (width 0) (type default))
   )
@@
     (stroke (width 0) (type default))
   )
+  (wire (pts (xy 154.6098 71.0438) (xy 156.464 71.0438))
+    (stroke (width 0) (type default))
+  )
   (wire (pts (xy 175.768 81.026) (xy 189.484 81.026))
     (stroke (width 0) (type default))
@@
     (stroke (width 0) (type default))
   )
+  (wire (pts (xy 156.21 73.5838) (xy 156.21 81.026))
+    (stroke (width 0) (type default))
+  )
   (wire (pts (xy 48.8188 37.4396) (xy 55.5244 37.4396))
     (stroke (width 0) (type default))
@@
   )
   (wire (pts (xy 238.76 70.6374) (xy 244.4496 70.6374))
+    (stroke (width 0) (type default))
+  )
+  (wire (pts (xy 156.464 71.0438) (xy 156.464 65.532))
     (stroke (width 0) (type default))
   )
@@
       (effects (font (size 1.27 1.27)) (justify left))
     )
-    (property "Value" "C" (at 210.82 67.818 90)
+    (property "Value" "TBD" (at 210.82 67.818 90)
       (effects (font (size 1.27 1.27)) (justify left))
     )
@@
         (path "/1805b3c6-7591-4bf3-945c-2567f5d02294"
           (reference "H1") (unit 1)
-        )
-      )
-    )
-  )
-  (symbol (lib_id "Device:Crystal_GND23") (at 115.2906 72.4916 0) (unit 1)
-    (in_bom yes) (on_board yes) (dnp no)
-    (property "Reference" "Y1" (at 119.3038 68.1482 0)
-      (effects (font (size 1.27 1.27)))
-    )
-    (property "Value" "Crystal_GND23" (at 126.746 70.8407 0)
-      (effects (font (size 1.27 1.27)) hide)
-    )
-    (property "Footprint" "Crystal:Crystal_SMD_2016-4Pin_2.0x1.6mm" (at 115.2906 72.4916 0)
-      (effects (font (size 1.27 1.27)) hide)
-    )
-    (property "Datasheet" "~" (at 115.2906 72.4916 0)
-      (effects (font (size 1.27 1.27)) hide)
-    )
-    (pin "4")
-    (pin "3")
-    (pin "1")
-    (pin "2")
-    (instances
-      (project "NFC_Programmer"
-        (path "/1805b3c6-7591-4bf3-945c-2567f5d02294"
-          (reference "Y1") (unit 1)
         )
       )
@@
     )
   )
+  (symbol (lib_id "Device:Crystal_GND24") (at 115.2906 72.4916 0) (unit 1)
+    (in_bom yes) (on_board yes) (dnp no)
+    (property "Reference" "Y1" (at 118.8466 67.6148 0)
+      (effects (font (size 1.27 1.27)))
+    )
+    (property "Value" "Crystal_27.12MHz" (at 124.8918 77.089 0)
+      (effects (font (size 1.27 1.27)) hide)
+    )
+    (property "Footprint" "Crystal:Crystal_SMD_2016-4Pin_2.0x1.6mm" (at 115.2906 72.4916 0)
+      (effects (font (size 1.27 1.27)) hide)
+    )
+    (property "Datasheet" "https://www.mouser.mx/datasheet/2/122/ECX_1637B2-2400564.pdf" (at 115.2906 72.4916 0)
+      (effects (font (size 1.27 1.27)) hide)
+    )
+    (pin "2")
+    (pin "1")
+    (pin "4")
+    (pin "3")
+    (instances
+      (project "NFC_Programmer"
+        (path "/1805b3c6-7591-4bf3-945c-2567f5d02294"
+          (reference "Y1") (unit 1)
+        )
+      )
+    )
+  )
   (symbol (lib_id "power:GND") (at 115.2906 88.6206 0) (unit 1)
     (in_bom yes) (on_board yes) (dnp no) (fields_autoplaced)
@@
   )
   (symbol (lib_id "Connector:Conn_01x02_Pin") (at 241.2746 45.3898 270) (unit 1)
-    (in_bom yes) (on_board yes) (dnp no) (fields_autoplaced)
-    (property "Reference" "J2" (at 242.4938 44.7548 90)
+    (in_bom yes) (on_board yes) (dnp no)
+    (property "Reference" "J2" (at 235.3818 44.7548 90)
       (effects (font (size 1.27 1.27)) (justify left))
     )
     (property "Value" "Conn_01x02_Pin" (at 242.4938 47.2948 90)
-      (effects (font (size 1.27 1.27)) (justify left))
-    )
-    (property "Footprint" "Connector_PinHeader_2.00mm:PinHeader_1x02_P2.00mm_Vertical" (at 241.2746 45.3898 0)
+      (effects (font (size 1.27 1.27)) (justify left) hide)
+    )
+    (property "Footprint" "Connector_PinHeader_2.54mm:PinHeader_1x02_P2.54mm_Vertical" (at 241.2746 45.3898 0)
       (effects (font (size 1.27 1.27)) hide)
     )
@@
       (effects (font (size 1.27 1.27)) (justify left) hide)
     )
-    (property "Footprint" "Connector_PinHeader_2.00mm:PinHeader_1x08_P2.00mm_Vertical" (at 53.3146 142.9004 0)
+    (property "Footprint" "Connector_PinHeader_2.54mm:PinHeader_1x08_P2.54mm_Vertical" (at 53.3146 142.9004 0)
       (effects (font (size 1.27 1.27)) hide)
     )
@@
         )
       )
+    )
+  )
+  (symbol (lib_id "Connector:Conn_01x02_Pin") (at 149.5298 71.0438 0) (unit 1)
+    (in_bom yes) (on_board yes) (dnp no)
+    (property "Reference" "J3" (at 150.241 68.5546 0)
+      (effects (font (size 1.27 1.27)))
+    )
+    (property "Value" "Conn_01x02_Pin" (at 150.1648 68.1482 0)
+      (effects (font (size 1.27 1.27)) hide)
+    )
+    (property "Footprint" "Connector_PinHeader_2.54mm:PinHeader_1x02_P2.54mm_Vertical" (at 149.5298 71.0438 0)
+      (effects (font (size 1.27 1.27)) hide)
+    )
+    (property "Datasheet" "~" (at 149.5298 71.0438 0)
+      (effects (font (size 1.27 1.27)) hide)
+    )
+    (pin "2")
+    (pin "1")
+    (instances
+      (project "NFC_Programmer"
+        (path "/1805b3c6-7591-4bf3-945c-2567f5d02294"
+          (reference "J3") (unit 1)
+        )
+      )
