File: hardware/PCB_Antena_IRIS/NFC_Programmer.kicad_sch (KiCad schematic)
At the start: 41 parts, among them J1 Conn_01x08, J2 Conn_01x02_Pin, U1 MFRC63002HN,151, Y1 Crystal_GND23

Commit message: Actualizacion
Parts:
- removed Y1: Crystal_GND23, Crystal:Crystal_SMD_2016-4Pin_2.0x1.6mm, symbol Device:Crystal_GND23
- added J3: Conn_01x02_Pin, Connector_PinHeader_2.54mm:PinHeader_1x02_P2.54mm_Vertical, symbol Connector:Conn_01x02_Pin
- added Y1: Crystal_GND24, symbol Device:Crystal_GND24
- J1: footprint Connector_PinHeader_2.00mm:PinHeader_1x08_P2.00mm_Vertical -> Connector_PinHeader_2.54mm:PinHeader_1x08_P2.54mm_Vertical
- J2: footprint Connector_PinHeader_2.00mm:PinHeader_1x02_P2.00mm_Vertical -> Connector_PinHeader_2.54mm:PinHeader_1x02_P2.54mm_Vertical
Connections:
- net GND: now also R1.1, Y1.2, Y1.4; no longer R1.2
- net PDOWN: now also R1.2; no longer R1.1
- net TX1: now also J3.1 (Pin_1)
- net TX2: now also J3.2 (Pin_2)
- net at C7.1, U1.19 (XTAL1): now also Y1.1
- net at C8.1, U1.20 (XTAL2): now also Y1.3
Other:
- note added: "MH, TP and PWR flags"
- note removed: "MH and PWR flags"
- moved on the sheet: C1, R1, TP1, TP2
