File: hardware/PCB_Antena_IRIS_2Vueltas/NFC_Programmer.kicad_pcb (KiCad board)
At the start: 2 copper layers, 40 x 56.1 mm, 40 parts, among them J1 Conn_01x08, J2 Conn_01x02_Pin, U1 MFRC63002HN,151, Y1 Crystal_GND23

Commit message: Actualizacion
Parts:
- added J3: Conn_01x02_Pin, Connector_PinHeader_2.54mm:PinHeader_1x02_P2.54mm_Vertical, F.Cu at (156.0, 102.5)
- J1: footprint Connector_PinHeader_2.00mm:PinHeader_1x08_P2.00mm_Vertical -> Connector_PinHeader_2.54mm:PinHeader_1x08_P2.54mm_Vertical
- J2: footprint Connector_PinHeader_2.00mm:PinHeader_1x02_P2.00mm_Vertical -> Connector_PinHeader_2.54mm:PinHeader_1x02_P2.54mm_Vertical
- Y1: value Crystal_GND23 -> Crystal_27.12MHz
- moved J1 0.20 mm to (137.7, 108.0)
- moved C7 0.06 mm to (137.1, 98.6)
- turned Y1 to -90 degrees
- renumbered SDA to TP1
Connections:
- Y1 pad 3: GND -> Net-(U1-XTAL2)
- Y1 pad 4: Net-(U1-XTAL2) -> GND
Routing:
- net /TX1: track 2.94 -> 23.2 mm, vias 0 -> 1
- net /TX2: track 2.36 -> 19.8 mm, vias 0 -> 1
- net GND: track 14.5 -> 16.9 mm, vias 269 -> 257
- net Net-(U1-XTAL1): track 4.49 -> 6.35 mm
- net /NSS: track 6.28 -> 7.83 mm
- net /IRQ: track 8.05 -> 9.56 mm
- net /MISO: track 4.89 -> 5.99 mm
- net +3V3: track 47.1 -> 48.1 mm
- net /SCK: track 4.31 -> 5.14 mm
- net /IFSEL1: track 14.8 -> 15.5 mm
- net /PDOWN: track 10.00 -> 10.6 mm
Other:
- board text added: "SDA"
