File: hardware/PCB_Antena_IRIS_2Vueltas/NFC_Programmer.kicad_sch (KiCad schematic)
At the start: 41 parts, among them J1 Conn_01x08, J2 Conn_01x02_Pin, U1 MFRC63002HN,151, Y1 Crystal_GND23

Commit message: Actualizacion
Parts:
- removed Y1: Crystal_GND23, Crystal:Crystal_SMD_2016-4Pin_2.0x1.6mm, symbol Device:Crystal_GND23
- added J3: Conn_01x02_Pin, Connector_PinHeader_2.54mm:PinHeader_1x02_P2.54mm_Vertical, symbol Connector:Conn_01x02_Pin
- added Y1: Crystal_27.12MHz, Crystal:Crystal_SMD_2016-4Pin_2.0x1.6mm, symbol Device:Crystal_GND24
- J1: footprint Connector_PinHeader_2.00mm:PinHeader_1x08_P2.00mm_Vertical -> Connector_PinHeader_2.54mm:PinHeader_1x08_P2.54mm_Vertical
- J2: footprint Connector_PinHeader_2.00mm:PinHeader_1x02_P2.00mm_Vertical -> Connector_PinHeader_2.54mm:PinHeader_1x02_P2.54mm_Vertical
Connections:
- net GND: now also Y1.2, Y1.4
- net TX1: now also J3.1 (Pin_1)
- net TX2: now also J3.2 (Pin_2)
- net at C7.1, U1.19 (XTAL1): now also Y1.1
- net at C8.1, U1.20 (XTAL2): now also Y1.3
Changed lines of the file:
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@@
+    (stroke (width 0) (type default))
+  )
+  (wire (pts (xy 155.1686 71.1962) (xy 156.464 71.1962))
     (stroke (width 0) (type default))
   )
@@
     (stroke (width 0) (type default))
   )
+  (wire (pts (xy 156.464 71.1962) (xy 156.464 65.532))
+    (stroke (width 0) (type default))
+  )
   (wire (pts (xy 252.8316 71.6026) (xy 248.4882 71.6026))
     (stroke (width 0) (type default))
@@
     (stroke (width 0) (type default))
   )
+  (wire (pts (xy 155.1686 73.7362) (xy 156.21 73.7362))
+    (stroke (width 0) (type default))
+  )
   (wire (pts (xy 244.3226 81.026) (xy 244.3226 79.2226))
     (stroke (width 0) (type default))
@@
   )
   (wire (pts (xy 27.686 74.8792) (xy 27.686 77.851))
+    (stroke (width 0) (type default))
+  )
+  (wire (pts (xy 156.21 73.7362) (xy 156.21 81.026))
     (stroke (width 0) (type default))
   )
@@
     )
   )
-  (symbol (lib_id "Device:Crystal_GND23") (at 115.2906 72.4916 0) (unit 1)
-    (in_bom yes) (on_board yes) (dnp no)
-    (property "Reference" "Y1" (at 119.3038 68.1482 0)
-      (effects (font (size 1.27 1.27)))
-    )
-    (property "Value" "Crystal_GND23" (at 126.746 70.8407 0)
-      (effects (font (size 1.27 1.27)) hide)
-    )
-    (property "Footprint" "Crystal:Crystal_SMD_2016-4Pin_2.0x1.6mm" (at 115.2906 72.4916 0)
-      (effects (font (size 1.27 1.27)) hide)
-    )
-    (property "Datasheet" "~" (at 115.2906 72.4916 0)
-      (effects (font (size 1.27 1.27)) hide)
-    )
-    (pin "4")
-    (pin "3")
-    (pin "1")
-    (pin "2")
-    (instances
-      (project "NFC_Programmer"
-        (path "/1805b3c6-7591-4bf3-945c-2567f5d02294"
-          (reference "Y1") (unit 1)
-        )
-      )
-    )
-  )
   (symbol (lib_id "Device:C") (at 189.484 69.342 0) (unit 1)
     (in_bom yes) (on_board yes) (dnp no)
@@
   (symbol (lib_id "Connector:TestPoint") (at 141.605 150.5966 0) (unit 1)
     (in_bom yes) (on_board yes) (dnp no) (fields_autoplaced)
-    (property "Reference" "TP1" (at 144.2466 146.0246 0)
-      (effects (font (size 1.27 1.27)) (justify left))
-    )
-    (property "Value" "TestPoint" (at 144.2466 148.5646 0)
+    (property "Reference" "TP1" (at 143.51 146.0246 0)
+      (effects (font (size 1.27 1.27)) (justify left))
+    )
+    (property "Value" "TestPoint" (at 143.51 148.5646 0)
       (effects (font (size 1.27 1.27)) (justify left))
     )
@@
     )
     (property "Value" "Conn_01x02_Pin" (at 242.4938 47.2948 90)
-      (effects (font (size 1.27 1.27)) (justify left))
-    )
-    (property "Footprint" "Connector_PinHeader_2.00mm:PinHeader_1x02_P2.00mm_Vertical" (at 241.2746 45.3898 0)
+      (effects (font (size 1.27 1.27)) (justify left) hide)
+    )
+    (property "Footprint" "Connector_PinHeader_2.54mm:PinHeader_1x02_P2.54mm_Vertical" (at 241.2746 45.3898 0)
       (effects (font (size 1.27 1.27)) hide)
     )
@@
         (path "/1805b3c6-7591-4bf3-945c-2567f5d02294"
           (reference "C6") (unit 1)
+        )
+      )
+    )
+  )
+  (symbol (lib_id "Device:Crystal_GND24") (at 115.2906 72.4916 0) (unit 1)
+    (in_bom yes) (on_board yes) (dnp no)
+    (property "Reference" "Y1" (at 119.38 68.0466 0)
+      (effects (font (size 1.27 1.27)))
+    )
+    (property "Value" "Crystal_27.12MHz" (at 125.603 70.8407 0)
+      (effects (font (size 1.27 1.27)) hide)
+    )
+    (property "Footprint" "Crystal:Crystal_SMD_2016-4Pin_2.0x1.6mm" (at 115.2906 72.4916 0)
+      (effects (font (size 1.27 1.27)) hide)
+    )
+    (property "Datasheet" "https://www.mouser.mx/datasheet/2/122/ECX_1637B2-2400564.pdf" (at 115.2906 72.4916 0)
+      (effects (font (size 1.27 1.27)) hide)
+    )
+    (pin "4")
+    (pin "1")
+    (pin "2")
+    (pin "3")
+    (instances
+      (project "NFC_Programmer"
+        (path "/1805b3c6-7591-4bf3-945c-2567f5d02294"
+          (reference "Y1") (unit 1)
         )
       )
@@
       (effects (font (size 1.27 1.27)) (justify left) hide)
     )
-    (property "Footprint" "Connector_PinHeader_2.00mm:PinHeader_1x08_P2.00mm_Vertical" (at 53.3146 142.9004 0)
+    (property "Footprint" "Connector_PinHeader_2.54mm:PinHeader_1x08_P2.54mm_Vertical" (at 53.3146 142.9004 0)
       (effects (font (size 1.27 1.27)) hide)
     )
@@
         )
       )
+    )
+  )
+  (symbol (lib_id "Connector:Conn_01x02_Pin") (at 150.0886 71.1962 0) (unit 1)
+    (in_bom yes) (on_board yes) (dnp no) (fields_autoplaced)
+    (property "Reference" "J3" (at 150.7236 68.7832 0)
+      (effects (font (size 1.27 1.27)))
+    )
+    (property "Value" "Conn_01x02_Pin" (at 151.9936 69.977 90)
+      (effects (font (size 1.27 1.27)) (justify left) hide)
+    )
+    (property "Footprint" "Connector_PinHeader_2.54mm:PinHeader_1x02_P2.54mm_Vertical" (at 150.0886 71.1962 0)
+      (effects (font (size 1.27 1.27)) hide)
+    )
+    (property "Datasheet" "~" (at 150.0886 71.1962 0)
+      (effects (font (size 1.27 1.27)) hide)
+    )
+    (pin "2")
+    (pin "1")
+    (instances
+      (project "NFC_Programmer"
+        (path "/1805b3c6-7591-4bf3-945c-2567f5d02294"
+          (reference "J3") (unit 1)
+        )
+      )
