File: hardware/PCB_IRIS_CAMBIO_PISTAS/NFC_Programmer.kicad_sch (KiCad schematic)
At the start: 41 parts, among them J1 Conn_01x08, J2 Conn_01x02_Pin, U1 MFRC63002HN,151, Y1 Crystal_GND23

Commit message: Actualizacion
Parts:
- removed Y1: Crystal_GND23, Crystal:Crystal_SMD_2016-4Pin_2.0x1.6mm, symbol Device:Crystal_GND23
- added J3: Conn_01x02_Pin, Connector_PinHeader_2.54mm:PinHeader_1x02_P2.54mm_Vertical, symbol Connector:Conn_01x02_Pin
- added Y1: Crystal_GND24, Crystal:Crystal_SMD_2016-4Pin_2.0x1.6mm, symbol Device:Crystal_GND24
- J1: footprint Connector_PinHeader_2.00mm:PinHeader_1x08_P2.00mm_Vertical -> Connector_PinHeader_2.54mm:PinHeader_1x08_P2.54mm_Vertical
- J2: footprint Connector_PinHeader_2.00mm:PinHeader_1x02_P2.00mm_Vertical -> Connector_PinHeader_2.54mm:PinHeader_1x02_P2.54mm_Vertical
Connections:
- net GND: now also Y1.2, Y1.4
- net TX1: now also J3.1 (Pin_1)
- net TX2: now also J3.2 (Pin_2)
- net at C7.1, U1.19 (XTAL1): now also Y1.1
- net at C8.1, U1.20 (XTAL2): now also Y1.3
Changed lines of the file:
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@@
+    (stroke (width 0) (type default))
+  )
+  (wire (pts (xy 155.3718 70.5358) (xy 156.464 70.5358))
     (stroke (width 0) (type default))
   )
@@
     (stroke (width 0) (type default))
   )
+  (wire (pts (xy 114.808 67.4116) (xy 115.2906 67.4116))
+    (stroke (width 0) (type default))
+  )
   (wire (pts (xy 90.3224 82.5246) (xy 90.3224 82.4992))
     (stroke (width 0) (type default))
@@
     (stroke (width 0) (type default))
   )
+  (wire (pts (xy 155.3718 73.0758) (xy 156.21 73.0758))
+    (stroke (width 0) (type default))
+  )
   (wire (pts (xy 244.3226 81.026) (xy 244.3226 79.2226))
     (stroke (width 0) (type default))
@@
     (stroke (width 0) (type default))
   )
+  (wire (pts (xy 156.464 70.5358) (xy 156.464 65.532))
+    (stroke (width 0) (type default))
+  )
   (wire (pts (xy 232.918 65.532) (xy 240.6396 65.532))
     (stroke (width 0) (type default))
@@
     (stroke (width 0) (type default))
   )
+  (wire (pts (xy 156.21 73.0758) (xy 156.21 81.026))
+    (stroke (width 0) (type default))
+  )
   (wire (pts (xy 241.2746 50.4698) (xy 241.2746 53.721))
     (stroke (width 0) (type default))
   )
   (wire (pts (xy 218.948 73.152) (xy 218.948 72.898))
-    (stroke (width 0) (type default))
-  )
-  (wire (pts (xy 114.808 67.4116) (xy 115.2906 67.4116))
     (stroke (width 0) (type default))
   )
@@
     )
   )
+  (symbol (lib_id "Device:Crystal_GND24") (at 115.2906 72.4916 0) (unit 1)
+    (in_bom yes) (on_board yes) (dnp no)
+    (property "Reference" "Y1" (at 118.8212 67.818 0)
+      (effects (font (size 1.27 1.27)))
+    )
+    (property "Value" "Crystal_GND24" (at 125.7554 70.8407 0)
+      (effects (font (size 1.27 1.27)) hide)
+    )
+    (property "Footprint" "Crystal:Crystal_SMD_2016-4Pin_2.0x1.6mm" (at 115.2906 72.4916 0)
+      (effects (font (size 1.27 1.27)) hide)
+    )
+    (property "Datasheet" "https://www.mouser.mx/datasheet/2/122/ECX_1637B2-2400564.pdf" (at 115.2906 72.4916 0)
+      (effects (font (size 1.27 1.27)) hide)
+    )
+    (pin "3")
+    (pin "2")
+    (pin "4")
+    (pin "1")
+    (instances
+      (project "NFC_Programmer"
+        (path "/1805b3c6-7591-4bf3-945c-2567f5d02294"
+          (reference "Y1") (unit 1)
+        )
+      )
+    )
+  )
   (symbol (lib_id "Device:R") (at 168.91 101.346 0) (unit 1)
     (in_bom yes) (on_board yes) (dnp no) (fields_autoplaced)
@@
         (path "/1805b3c6-7591-4bf3-945c-2567f5d02294"
           (reference "TP2") (unit 1)
-        )
-      )
-    )
-  )
-  (symbol (lib_id "Device:Crystal_GND23") (at 115.2906 72.4916 0) (unit 1)
-    (in_bom yes) (on_board yes) (dnp no)
-    (property "Reference" "Y1" (at 119.3038 68.1482 0)
-      (effects (font (size 1.27 1.27)))
-    )
-    (property "Value" "Crystal_GND23" (at 126.746 70.8407 0)
-      (effects (font (size 1.27 1.27)) hide)
-    )
-    (property "Footprint" "Crystal:Crystal_SMD_2016-4Pin_2.0x1.6mm" (at 115.2906 72.4916 0)
-      (effects (font (size 1.27 1.27)) hide)
-    )
-    (property "Datasheet" "~" (at 115.2906 72.4916 0)
-      (effects (font (size 1.27 1.27)) hide)
-    )
-    (pin "4")
-    (pin "3")
-    (pin "1")
-    (pin "2")
-    (instances
-      (project "NFC_Programmer"
-        (path "/1805b3c6-7591-4bf3-945c-2567f5d02294"
-          (reference "Y1") (unit 1)
         )
       )
@@
   )
   (symbol (lib_id "Connector:Conn_01x02_Pin") (at 241.2746 45.3898 270) (unit 1)
-    (in_bom yes) (on_board yes) (dnp no) (fields_autoplaced)
-    (property "Reference" "J2" (at 242.4938 44.7548 90)
+    (in_bom yes) (on_board yes) (dnp no)
+    (property "Reference" "J2" (at 236.0168 44.6786 90)
       (effects (font (size 1.27 1.27)) (justify left))
     )
     (property "Value" "Conn_01x02_Pin" (at 242.4938 47.2948 90)
-      (effects (font (size 1.27 1.27)) (justify left))
-    )
-    (property "Footprint" "Connector_PinHeader_2.00mm:PinHeader_1x02_P2.00mm_Vertical" (at 241.2746 45.3898 0)
-      (effects (font (size 1.27 1.27)) hide)
-    )
-    (property "Datasheet" "~" (at 241.2746 45.3898 0)
+      (effects (font (size 1.27 1.27)) (justify left) hide)
+    )
+    (property "Footprint" "Connector_PinHeader_2.54mm:PinHeader_1x02_P2.54mm_Vertical" (at 241.2746 45.3898 0)
+      (effects (font (size 1.27 1.27)) hide)
+    )
+    (property "Datasheet" "" (at 241.2746 45.3898 0)
       (effects (font (size 1.27 1.27)) hide)
     )
@@
         (path "/1805b3c6-7591-4bf3-945c-2567f5d02294"
           (reference "#PWR09") (unit 1)
+        )
+      )
+    )
+  )
+  (symbol (lib_id "Connector:Conn_01x02_Pin") (at 150.2918 70.5358 0) (unit 1)
+    (in_bom yes) (on_board yes) (dnp no)
+    (property "Reference" "J3" (at 148.9964 68.9864 0)
+      (effects (font (size 1.27 1.27)) (justify left))
+    )
+    (property "Value" "Conn_01x02_Pin" (at 152.1968 69.3166 90)
+      (effects (font (size 1.27 1.27)) (justify left) hide)
+    )
+    (property "Footprint" "Connector_PinHeader_2.54mm:PinHeader_1x02_P2.54mm_Vertical" (at 150.2918 70.5358 0)
+      (effects (font (size 1.27 1.27)) hide)
+    )
+    (property "Datasheet" "" (at 150.2918 70.5358 0)
+      (effects (font (size 1.27 1.27)) hide)
+    )
+    (pin "2")
+    (pin "1")
+    (instances
+      (project "NFC_Programmer"
+        (path "/1805b3c6-7591-4bf3-945c-2567f5d02294"
+          (reference "J3") (unit 1)
         )
       )
@@
       (effects (font (size 1.27 1.27)) (justify left) hide)
     )
-    (property "Footprint" "Connector_PinHeader_2.00mm:PinHeader_1x08_P2.00mm_Vertical" (at 53.3146 142.9004 0)
-      (effects (font (size 1.27 1.27)) hide)
-    )
+    (property "Footprint" "Connector_PinHeader_2.54mm:PinHeader_1x08_P2.54mm_Vertical" (at 53.3146 142.9004 0)
+      (effects (font (size 1.27 1.27)) hide)
+    )
